File: BatteryBoost.kicad_pcb (KiCad board)
At the start: 2 copper layers, 80 x 40 mm, 44 parts, among them J1 Mounting Hole, J2 Mounting Hole, J3 Mounting Hole, J4 Mounting Hole, J5 USB_B_Micro, J6 Battery, J7 Output, Q1 -40V 7.5A 2.5V @ 250uA 40mΩ @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, Q2 -40V 7.5A 40mΩ @ 6A, Q4 20V 7.5A 24mΩ @ 2.5Vgs, SW1 SW_SPDT, U1 SP34063AEN, U2 TP4056, U3 AP9101CK6

Commit message: Add artwork and finalize layout
Parts:
- turned R11 to 180 degrees
Routing:
- net /Raw_Batt_-: track 35.7 -> 74.8 mm, vias 1 -> 2
- net SMPS_Output: track 0.00 -> 24.1 mm, vias 0 -> 2
- net Net-(R11-Pad2): track 12.8 -> 0.00 mm
- net Net-(R11-Pad1): track 0.00 -> 12.8 mm
Other:
- board text added: "BAT"
- board text added: "OUT"
